Commit message: Camera added to Gazebo

File: src/crawler_description/urdf/crawler.urdf.xacro (robot description, xacro)
@@ -122,4 +122,5 @@
   <link name="camera_front_link">
     <visual>
+      <origin xyz="0 0 0" rpy="1.57 0 1.57"/>
       <geometry>
         <mesh filename="package://crawler_description/meshes/camera.stl" scale="0.001 0.001 0.001"/>
@@ -137,6 +138,7 @@
     </inertial>
   </link>
-  <link name="camera_back_link">
-    <visual>
+<link name="camera_back_link">
+    <visual>
+      <origin xyz="0 0 0" rpy="-1.57 0 1.57"/>
       <geometry>
         <mesh filename="package://crawler_description/meshes/camera.stl" scale="0.001 0.001 0.001"/>
@@ -153,5 +155,5 @@
       <inertia ixx="0.00001" ixy="0.0" ixz="0.0" iyy="0.00003" iyz="0.0" izz="0.00003"/>
     </inertial>
-  </link>
+</link>
   <link name="lidar_link">
     <visual>
@@ -224,10 +226,10 @@
     <parent link="base_link"/>
     <child link="camera_front_link"/>
-    <origin xyz="0.210 0.0514 0.01" rpy="1.57 0 1.57"/>
+    <origin xyz="0.210 0.0514 0.01" rpy="0 0 0"/>
   </joint>
   <joint name="camera_back_joint" type="fixed">
     <parent link="base_link"/>
     <child link="camera_back_link"/>
-    <origin xyz="-0.210 0.0513 0.01" rpy="-1.57 0 1.57"/>
+    <origin xyz="-0.210 0.0513 0.01" rpy="0 0 3.14"/>
   </joint>
   <joint name="lidar_joint" type="fixed">

File: src/crawler_description/urdf/crawler_gazebo.xacro (robot description, xacro)
@@ -37,3 +37,53 @@
         <fdir1>0 1 0</fdir1>
     </gazebo>
+    <gazebo reference="camera_front_link">
+        <sensor name="camera_front_sensor" type="camera">
+            <pose>0 0 0 0 0 0</pose>
+            <visualize>true</visualize>
+            <update_rate>10.0</update_rate>
+            <plugin name="camera_front_controller" filename="libgazebo_ros_camera.so">
+                <frame_name>camera_front_link</frame_name>
+            </plugin>
+        </sensor>
+    </gazebo>
+    <gazebo reference="camera_back_link">
+        <sensor name="camera_back_sensor" type="camera">
+            <pose>0 0 0 0 0 0</pose>
+            <visualize>true</visualize>
+            <update_rate>10.0</update_rate>
+            <plugin name="camera_back_controller" filename="libgazebo_ros_camera.so">
+                <frame_name>camera_back_link</frame_name>
+            </plugin>
+        </sensor>
+    </gazebo>
+    <gazebo reference="lidar_link">
+        <sensor name="lidar" type="ray">
+          <pose>0 0 0 0 0 0</pose>
+          <visualize>true</visualize>
+          <update_rate>10.0</update_rate>
+          <ray>
+            <scan>
+              <horizontal>
+                <samples>720</samples>
+                <resolution>1</resolution>
+                <min_angle>-1.047</min_angle>
+                <max_angle>1.047</max_angle>
+              </horizontal>
+            </scan>
+            <range>
+              <min>0.1</min>
+              <max>10.0</max>
+              <resolution>0.01</resolution>
+            </range>
+            <noise>
+              <type>gaussian</type>
+              <mean>0.0</mean>
+              <stddev>0.01</stddev>
+            </noise>
+          </ray>
+          <plugin name="front_lidar_plugin" filename="libgazebo_ros_ray_sensor.so">
+            <update_rate>10.0 </update_rate>
+          </plugin>
+        </sensor>
+    </gazebo>
 </robot>

Commit message: LaserScan Added

File: src/crawler_description/urdf/crawler.urdf.xacro (robot description, xacro)
@@ -158,4 +158,5 @@
   <link name="lidar_link">
     <visual>
+    <origin xyz="0 -0.02065 0.0046" rpy="1.57 0 0"/>
       <geometry>
         <mesh filename="package://crawler_description/meshes/lidar.stl" scale="0.001 0.001 0.001"/>
@@ -236,5 +237,5 @@
     <parent link="base_link"/>
     <child link="lidar_link"/>
-    <origin xyz="0.173 0.0 0.035" rpy="1.57 0 0"/>
+    <origin xyz="0.173 0.0 0.035" rpy="0 0 0"/>
   </joint>
   <joint name="probe_holder_joint" type="fixed">

File: src/crawler_description/urdf/crawler_gazebo.xacro (robot description, xacro)
@@ -59,5 +59,5 @@
     <gazebo reference="lidar_link">
         <sensor name="lidar" type="ray">
-          <pose>0 0 0 0 0 0</pose>
+          <pose>-1.57 0 0 0 0 0</pose>
           <visualize>true</visualize>
           <update_rate>10.0</update_rate>

Commit message: Control Added

File: src/crawler_description/urdf/crawler.urdf.xacro (robot description, xacro)
@@ -2,4 +2,5 @@
 <robot name="crawler" xmlns:xacro="http://www.ros.org/wiki/xacro">
   <xacro:include filename="$(find crawler_description)/urdf/crawler_gazebo.xacro" />
+  <xacro:include filename="$(find crawler_description)/urdf/crawler_ros2_control.xacro" />
     <material name="body_grey">
     <color rgba="0.35 0.35 0.38 1.0"/>
@@ -202,4 +203,5 @@
     <axis xyz="0 1 0"/>
     <dynamics damping="0.2" friction="0.1"/>
+    <limit effort="10" velocity="1.0"/>
   </joint>
   <joint name="front_left_wheel_joint" type="continuous">
@@ -209,4 +211,5 @@
     <axis xyz="0 1 0"/>
     <dynamics damping="0.2" friction="0.1"/>
+    <limit effort="10" velocity="1.0"/>
   </joint>
   <joint name="rear_right_wheel_joint" type="continuous">
@@ -216,4 +219,5 @@
     <axis xyz="0 1 0"/>
     <dynamics damping="0.2" friction="0.1"/>
+    <limit effort="10" velocity="1.0"/>
   </joint>
   <joint name="rear_left_wheel_joint" type="continuous">

File: src/crawler_description/urdf/crawler_gazebo.xacro (robot description, xacro)
@@ -87,3 +87,8 @@
         </sensor>
     </gazebo>
+    <gazebo>
+        <plugin name="gazebo_ros2_control" filename="libgazebo_ros2_control.so">
+            <parameters>$(find crawler_controller)/config/crawler_controllers.yaml</parameters>
+        </plugin>
+    </gazebo>
 </robot>

Commit message: Error in crawler.urdf.xacro corrected

File: src/crawler_description/urdf/crawler.urdf.xacro (robot description, xacro)
@@ -203,5 +203,5 @@
     <axis xyz="0 1 0"/>
     <dynamics damping="0.2" friction="0.1"/>
-    <limit effort="10" velocity="1.0"/>
+    <limit effort="10" velocity="2.0"/>
   </joint>
   <joint name="front_left_wheel_joint" type="continuous">
@@ -211,5 +211,5 @@
     <axis xyz="0 1 0"/>
     <dynamics damping="0.2" friction="0.1"/>
-    <limit effort="10" velocity="1.0"/>
+    <limit effort="10" velocity="2.0"/>
   </joint>
   <joint name="rear_right_wheel_joint" type="continuous">
@@ -219,5 +219,5 @@
     <axis xyz="0 1 0"/>
     <dynamics damping="0.2" friction="0.1"/>
-    <limit effort="10" velocity="1.0"/>
+    <limit effort="10" velocity="2.0"/>
   </joint>
   <joint name="rear_left_wheel_joint" type="continuous">
@@ -227,4 +227,5 @@
     <axis xyz="0 1 0"/>
     <dynamics damping="0.2" friction="0.1"/>
+    <limit effort="10" velocity="2.0"/>
   </joint>
   <joint name="camera_front_joint" type="fixed">
